Commit message: Update many things

File: src/turtlebot3/turtlebot3_description/urdf/turtlebot3_burger.gazebo.xacro (robot description, xacro)
@@ -7,6 +7,6 @@
   </gazebo>
   <gazebo reference="wheel_left_link">
-    <mu1>0.1</mu1>
-    <mu2>0.1</mu2>
+    <mu1>1.0</mu1>
+    <mu2>1.0</mu2>
     <kp>500000.0</kp>
     <kd>10.0</kd>
@@ -17,6 +17,6 @@
   </gazebo>
   <gazebo reference="wheel_right_link">
-    <mu1>0.1</mu1>
-    <mu2>0.1</mu2>
+    <mu1>1.0</mu1>
+    <mu2>1.0</mu2>
     <kp>500000.0</kp>
     <kd>10.0</kd>
@@ -101,5 +101,5 @@
         <scan>
           <horizontal>
-            <samples>480</samples>
+            <samples>10</samples>
             <resolution>1</resolution>
             <min_angle>-1.74533</min_angle>

File: src/turtlebot3/turtlebot3_description/urdf/turtlebot3_burger.urdf.xacro (robot description, xacro)
@@ -4,5 +4,5 @@
   <xacro:include filename="$(find turtlebot3_description)/urdf/turtlebot3_burger.gazebo.xacro"/>
   <!-- scale 변수 추가 -->
-  <xacro:property name="mesh_scale" value="0.005 0.005 0.005" />
+  <xacro:property name="mesh_scale" value="0.001 0.001 0.001" />
   <link name="base_footprint"/>
   <joint name="base_joint" type="fixed">

File: src/turtlebot3/turtlebot3_description/urdf/turtlebot3_waffle.gazebo.xacro (robot description, xacro)
@@ -1,5 +1,5 @@
 <?xml version="1.0"?>
 <robot name="turtlebot3_waffle_sim" xmlns:xacro="http://ros.org/wiki/xacro">
-  <xacro:arg name="laser_visual"  default="false"/>
+  <xacro:arg name="laser_visual"  default="true"/>
   <xacro:arg name="camera_visual" default="false"/>
   <xacro:arg name="imu_visual"    default="false"/>
@@ -8,6 +8,6 @@
   </gazebo>
   <gazebo reference="wheel_left_link">
-    <mu1>0.1</mu1>
-    <mu2>0.1</mu2>
+    <mu1>10.0</mu1>
+    <mu2>10.0</mu2>
     <kp>500000.0</kp>
     <kd>10.0</kd>
@@ -18,6 +18,6 @@
   </gazebo>
   <gazebo reference="wheel_right_link">
-    <mu1>0.1</mu1>
-    <mu2>0.1</mu2>
+    <mu1>10.0</mu1>
+    <mu2>10.0</mu2>
     <kp>500000.0</kp>
     <kd>10.0</kd>
@@ -106,18 +106,19 @@
     <sensor type="ray" name="lds_lfcd_sensor">
       <pose>0 0 0 0 0 0</pose>
-      <visualize>$(arg laser_visual)</visualize>
+      <!-- original code : <visualize>$(arg laser_visual)</visualize> -->
+      <visualize>true</visualize>
       <update_rate>5</update_rate>
       <ray>
         <scan>
           <horizontal>
-            <samples>360</samples>
+            <samples>10</samples>
             <resolution>1</resolution>
-            <min_angle>0.0</min_angle>
-            <max_angle>6.28319</max_angle>
+            <min_angle>-1.74533</min_angle>
+            <max_angle>1.74533</max_angle>
           </horizontal>
         </scan>
         <range>
           <min>0.120</min>
-          <max>3.5</max>
+          <max>4.0</max>
           <resolution>0.015</resolution>
         </range>
@@ -133,4 +134,15 @@
       </plugin>
     </sensor>
+  </gazebo>
+  <!-- Ground Truth Pose -->
+  <gazebo>
+    <plugin name="gazebo_ros_p3d" filename="libgazebo_ros_p3d.so">
+      <alwaysOn>true</alwaysOn>
+      <updateRate>30.0</updateRate>
+      <bodyName>base_footprint</bodyName>
+      <topicName>ground_truth_pose</topicName>
+      <gaussianNoise>0.0</gaussianNoise>
+      <frameName>map</frameName>
+    </plugin>
   </gazebo>
   <gazebo reference="camera_rgb_frame">

File: src/turtlebot3/turtlebot3_description/urdf/turtlebot3_waffle_pi.gazebo.xacro (robot description, xacro)
@@ -1,5 +1,5 @@
 <?xml version="1.0"?>
 <robot name="turtlebot3_waffle_pi_sim" xmlns:xacro="http://ros.org/wiki/xacro">
-  <xacro:arg name="laser_visual"  default="false"/>
+  <xacro:arg name="laser_visual"  default="true"/>
   <xacro:arg name="camera_visual" default="false"/>
   <xacro:arg name="imu_visual"    default="false"/>
@@ -8,6 +8,6 @@
   </gazebo>
   <gazebo reference="wheel_left_link">
-    <mu1>0.1</mu1>
-    <mu2>0.1</mu2>
+    <mu1>10.0</mu1>
+    <mu2>10.0</mu2>
     <kp>500000.0</kp>
     <kd>10.0</kd>
@@ -18,6 +18,6 @@
   </gazebo>
   <gazebo reference="wheel_right_link">
-    <mu1>0.1</mu1>
-    <mu2>0.1</mu2>
+    <mu1>10.0</mu1>
+    <mu2>10.0</mu2>
     <kp>500000.0</kp>
     <kd>10.0</kd>
@@ -111,13 +111,13 @@
         <scan>
           <horizontal>
-            <samples>360</samples>
+            <samples>10</samples>
             <resolution>1</resolution>
-            <min_angle>0.0</min_angle>
-            <max_angle>6.28319</max_angle>
+            <min_angle>-1.74533</min_angle>
+            <max_angle>1.74533</max_angle>
           </horizontal>
         </scan>
         <range>
           <min>0.120</min>
-          <max>3.5</max>
+          <max>4.0</max>
           <resolution>0.015</resolution>
         </range>
@@ -133,4 +133,15 @@
       </plugin>
     </sensor>
+  </gazebo>
+  <!-- Ground Truth Pose -->
+  <gazebo>
+    <plugin name="gazebo_ros_p3d" filename="libgazebo_ros_p3d.so">
+      <alwaysOn>true</alwaysOn>
+      <updateRate>30.0</updateRate>
+      <bodyName>base_footprint</bodyName>
+      <topicName>ground_truth_pose</topicName>
+      <gaussianNoise>0.0</gaussianNoise>
+      <frameName>map</frameName>
+    </plugin>
   </gazebo>
 <!--link : https://www.raspberrypi.org/documentation/hardware/camera/-->
